File: PCB/Multiplex/Multiplex.sch (KiCad schematic (older format))
At the start: 16 parts, among them J1+1 Power, J1-1 Power, J2+1 I2C, J2-1 I2C, J3 Signal, J4 Track, U1 PIC16F1503-IP, U2 MOC3041M

Commit message: .gitignore angepasst PCB Dateien hinzugefügt Can2Rest Webservice hinzugefügt
Parts:
- R5: footprint Resistor_THT:R_Axial_DIN0204_L3.6mm_D1.6mm_P7.62mm_Horizontal -> Resistor_THT:R_Axial_DIN0207_L6.3mm_D2.5mm_P10.16mm_Horizontal
Connections:
- net +5V: now reaches J1+1.1 (Pin_1), J1-1.1 (Pin_1), U1.1 (VDD)
- net GND: now reaches J1+1.2 (Pin_2), J1-1.2 (Pin_2), JP1.1 (A), JP2.1 (A), JP3.1 (A), U1.14 (VSS), U2.2
- net at U2.4: now also J4.2 (Pin_2); no longer J4.1 (Pin_1)
- net at U2.6: now also J4.1 (Pin_1); no longer J4.2 (Pin_2)
Changed lines of the file:
@@
 $EndComp
 Wire Wire Line
-	5650 2650 1000 2650
+	5650 2650 4025 2650
 Wire Wire Line
 	1000 2650 1000 3325
@@
 F 0 "R5" H 3720 3871 50  0000 L CNN
 F 1 "150" H 3720 3780 50  0000 L CNN
-F 2 "Resistor_THT:R_Axial_DIN0204_L3.6mm_D1.6mm_P7.62mm_Horizontal" V 3580 3825 50  0001 C CNN
+F 2 "Resistor_THT:R_Axial_DIN0207_L6.3mm_D2.5mm_P10.16mm_Horizontal" V 3580 3825 50  0001 C CNN
 F 3 "~" H 3650 3825 50  0001 C CNN
 	1    3650 3825
@@
 Connection ~ 3650 4775
 Wire Wire Line
-	3650 4775 5675 4775
+	3650 4775 3925 4775
 Wire Wire Line
 	2825 4300 3050 4300
@@
 L Connector_Generic:Conn_01x02 J4
 U 1 1 5E9FA994
-P 2625 4400
-F 0 "J4" H 2713 4314 50  0000 L CNN
-F 1 "Track" H 2713 4223 50  0000 L CNN
-F 2 "Connector_PinSocket_2.54mm:PinSocket_1x02_P2.54mm_Horizontal" H 2625 4400 50  0001 C CNN
-F 3 "~" H 2625 4400 50  0001 C CNN
-	1    2625 4400
-	-1   0    0    1
-$EndComp
+P 2625 4300
+F 0 "J4" H 2713 4214 50  0000 L CNN
+F 1 "Track" H 2713 4123 50  0000 L CNN
+F 2 "Connector_PinSocket_2.54mm:PinSocket_1x02_P2.54mm_Horizontal" H 2625 4300 50  0001 C CNN
+F 3 "~" H 2625 4300 50  0001 C CNN
+	1    2625 4300
+	-1   0    0    -1
+$EndComp
+$Comp
+L power:GND #PWR?
+U 1 1 5ED5824C
+P 3925 4775
+F 0 "#PWR?" H 3925 4525 50  0001 C CNN
+F 1 "GND" H 3930 4602 50  0000 C CNN
+F 2 "" H 3925 4775 50  0001 C CNN
+F 3 "" H 3925 4775 50  0001 C CNN
+	1    3925 4775
+	1    0    0    -1
+$EndComp
+Connection ~ 3925 4775
+Wire Wire Line
+	3925 4775 5675 4775
+$Comp
+L power:+5V #PWR?
+U 1 1 5ED588EC
+P 4025 2650
+F 0 "#PWR?" H 4025 2500 50  0001 C CNN
+F 1 "+5V" H 4040 2823 50  0000 C CNN
+F 2 "" H 4025 2650 50  0001 C CNN
+F 3 "" H 4025 2650 50  0001 C CNN
+	1    4025 2650
+	1    0    0    -1
+$EndComp
+Connection ~ 4025 2650
+Wire Wire Line
+	4025 2650 1000 2650
 $EndSCHEMATC
