File: PCB/I2CMaster/I2CMaster.kicad_pcb (KiCad board)
At the start: 2 copper layers, 52.1 x 35.6 mm, 20 parts, among them U1 PIC18F26K83-xSP, U2 MCP2561-E-P

Commit message: First try
Parts:
- added R4: 1600, Resistor_SMD:R_0603_1608Metric_Pad1.05x0.95mm_HandSolder, B.Cu at (350.5, 261.6)
- added R5: 1600, Resistor_SMD:R_0603_1608Metric_Pad1.05x0.95mm_HandSolder, B.Cu at (350.5, 259.1)
Connections:
- CAN-BUS1 pad 1: Net-(CAN-BUS1-Pad1) -> unconnected-(CAN-BUS1-Pin_1-Pad1)
- U1 pad 1: Net-(U1-Pad1) -> unconnected-(U1-VPP/~{MCLR}/RE3-Pad1)
- U1 pad 11: Net-(U1-Pad11) -> unconnected-(U1-RC0/SOSCO-Pad11)
- U1 pad 12: Net-(U1-Pad12) -> unconnected-(U1-RC1/SOSCI-Pad12)
- U1 pad 13: Net-(U1-Pad13) -> unconnected-(U1-RC2-Pad13)
- U1 pad 16: Net-(U1-Pad16) -> unconnected-(U1-RC5-Pad16)
- U1 pad 17: Net-(U1-Pad17) -> unconnected-(U1-RC6-Pad17)
- U1 pad 18: Net-(U1-Pad18) -> unconnected-(U1-RC7-Pad18)
- U1 pad 21: Net-(U1-Pad21) -> unconnected-(U1-RB0-Pad21)
- U1 pad 22: Net-(U1-Pad22) -> unconnected-(U1-RB1-Pad22)
- U1 pad 25: Net-(U1-Pad25) -> unconnected-(U1-RB4-Pad25)
- U1 pad 26: Net-(U1-Pad26) -> unconnected-(U1-RB5-Pad26)
- U1 pad 28: Net-(U1-Pad28) -> unconnected-(U1-ICSPDAT/RB7-Pad28)
Routing:
- net Net-(I2C1-Pin_2): track 14.9 -> 49.7 mm
- net Net-(I2C1-Pin_1): track 4.05 -> 34.5 mm
- net +5V: track 83.9 -> 93.7 mm
Other:
- net class Default removed
- board text added: "CAN to I2C Interface ©2021 Dominik Föhl"
- board text removed: "CAN to I2C Interface ©2020 Dominik Föhl"
