File: PCB/I2CMaster/I2CMaster.sch (KiCad schematic (older format))
At the start: 20 parts, among them U1 PIC18F26K83-xSP, U2 MCP2561-E-P

Commit message: First try
Parts:
- added R4, R5: 1600, Resistor_SMD:R_0603_1608Metric_Pad1.05x0.95mm_HandSolder, symbol Device:R
Connections:
- net GND: now also R4.2, R5.2
- net at I2C1.1 (Pin_1), U1.15 (RC4): now also R5.1
- net at I2C1.2 (Pin_2), U1.14 (RC3): now also R4.1
Changed lines of the file:
@@
 $EndComp
 Wire Wire Line
-	7875 4625 8775 4625
+	7875 4625 8225 4625
 Wire Wire Line
 	8775 4625 8775 2450
 Wire Wire Line
-	7875 4525 8675 4525
+	7875 4525 8025 4525
 Wire Wire Line
 	8675 4525 8675 2575
@@
 Connection ~ 6375 4925
 $Comp
-L power:+5V #PWR?
+L power:+5V #PWR0103
 U 1 1 5EDCC146
 P 4700 4325
-F 0 "#PWR?" H 4700 4175 50  0001 C CNN
+F 0 "#PWR0103" H 4700 4175 50  0001 C CNN
 F 1 "+5V" H 4715 4498 50  0000 C CNN
 F 2 "" H 4700 4325 50  0001 C CNN
@@
 Wire Wire Line
 	4700 4325 5725 4325
+$Comp
+L power:GND #PWR0104
+U 1 1 60B80F68
+P 8225 4925
+F 0 "#PWR0104" H 8225 4675 50  0001 C CNN
+F 1 "GND" H 8230 4752 50  0000 C CNN
+F 2 "" H 8225 4925 50  0001 C CNN
+F 3 "" H 8225 4925 50  0001 C CNN
+	1    8225 4925
+	1    0    0    -1
+$EndComp
+$Comp
+L Device:R R5
+U 1 1 60B81F54
+P 8225 4775
+F 0 "R5" H 8295 4821 50  0000 L CNN
+F 1 "1600" H 8295 4730 50  0000 L CNN
+F 2 "Resistor_SMD:R_0603_1608Metric_Pad1.05x0.95mm_HandSolder" V 8155 4775 50  0001 C CNN
+F 3 "~" H 8225 4775 50  0001 C CNN
+	1    8225 4775
+	1    0    0    -1
+$EndComp
+Connection ~ 8225 4625
+Wire Wire Line
+	8225 4625 8775 4625
+$Comp
+L Device:R R4
+U 1 1 60B828C7
+P 8025 4675
+F 0 "R4" H 8095 4721 50  0000 L CNN
+F 1 "1600" H 8095 4630 50  0000 L CNN
+F 2 "Resistor_SMD:R_0603_1608Metric_Pad1.05x0.95mm_HandSolder" V 7955 4675 50  0001 C CNN
+F 3 "~" H 8025 4675 50  0001 C CNN
+	1    8025 4675
+	1    0    0    -1
+$EndComp
+Connection ~ 8025 4525
+Wire Wire Line
+	8025 4525 8675 4525
+Wire Wire Line
+	8225 4925 8025 4925
+Wire Wire Line
+	8025 4925 8025 4825
+Connection ~ 8225 4925
 $EndSCHEMATC
