File: PCB/OptokopplerInput/OptokopplerInput.kicad_pcb (KiCad board)
At the start: 2 copper layers, 66 x 41.3 mm, 23 parts, among them J1+1 Power, J1-1 Power, J2+1 I2C, J2-1 I2C, J3 Screw_Terminal_01x12, U1 PIC16F1503-IP, U2 LTV-825, U3 LTV-845

Commit message: First try
Routing:
- net GND: track 23.5 -> 0.00 mm
Changed lines of the file:
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@@
   (segment (start 139.065 112.235) (end 139.065 106.68) (width 0.25) (layer "F.Cu") (net 12))
   (segment (start 139.065 106.68) (end 137.15 104.765) (width 0.25) (layer "F.Cu") (net 12))
-  (segment (start 184.005 107.805) (end 182.88 106.68) (width 0.25) (layer "F.Cu") (net 13))
-  (segment (start 177.8 106.68) (end 176.675 105.555) (width 0.25) (layer "F.Cu") (net 13))
-  (segment (start 179.375 105.105) (end 177.8 106.68) (width 0.25) (layer "F.Cu") (net 13))
-  (segment (start 186.835 107.805) (end 184.005 107.805) (width 0.25) (layer "F.Cu") (net 13))
-  (segment (start 187.96 106.68) (end 186.835 107.805) (width 0.25) (layer "F.Cu") (net 13))
-  (segment (start 176.675 105.555) (end 173.845 105.555) (width 0.25) (layer "F.Cu") (net 13))
-  (segment (start 186.385 105.105) (end 179.375 105.105) (width 0.25) (layer "F.Cu") (net 13))
-  (segment (start 187.96 106.68) (end 186.385 105.105) (width 0.25) (layer "F.Cu") (net 13))
-  (segment (start 173.845 105.555) (end 172.72 106.68) (width 0.25) (layer "F.Cu") (net 13))
   (segment (start 144.78 101.6) (end 149.86 106.68) (width 0.25) (layer "F.Cu") (net 14))
   (segment (start 140.97 101.6) (end 144.78 101.6) (width 0.25) (layer "F.Cu") (net 14))
