File: PCB/OptokopplerOutput/OptokopplerOutput.kicad_pcb (KiCad board)
At the start: 2 copper layers, 48.3 x 40.6 mm, 16 parts, among them J1+1 Power, J1-1 Power, J2+1 I2C, J2-1 I2C, J3 Signal, J4 Track, U1 PIC16F1503-IP, U2 MOC3041M

Commit message: First try
Parts:
- removed J3: Signal, Connector_PinHeader_2.00mm:PinHeader_2x02_P2.00mm_Horizontal
- removed J4: Track, Connector_PinHeader_2.54mm:PinHeader_1x02_P2.54mm_Horizontal
- added D1: 1N4001, Diode_SMD:D_SMB_Handsoldering, F.Cu at (166.4, 116.7)
- added D2: 1N4001, Diode_SMD:D_SMB_Handsoldering, F.Cu at (174.0, 119.4)
- added D3: 1N4001, Diode_SMD:D_SMB_Handsoldering, F.Cu at (176.5, 108.1)
- added D4: 1N4001, Diode_SMD:D_SMB_Handsoldering, F.Cu at (171.4, 108.1)
- added D5: 1N4001, Diode_SMD:D_SMB_Handsoldering, F.Cu at (191.8, 97.6)
- added D6: 1N4001, Diode_SMD:D_SMB_Handsoldering, F.Cu at (186.7, 97.6)
- added J1: Screw_Terminal_01x06, TerminalBlock_RND:TerminalBlock_RND_205-00236_1x06_P5.08mm_Horizontal, F.Cu at (190.5, 127.0)
- added J2: Screw_Terminal_01x06, TerminalBlock_RND:TerminalBlock_RND_205-00236_1x06_P5.08mm_Horizontal, F.Cu at (158.8, 127.0)
- added Q1: BD675, Package_TO_SOT_THT:TO-126-3_Vertical, F.Cu at (181.6, 110.5)
- added Q2: BD675, Package_TO_SOT_THT:TO-126-3_Vertical, F.Cu at (186.7, 110.5)
- added Q3: BD675, Package_TO_SOT_THT:TO-126-3_Vertical, F.Cu at (181.6, 119.4)
- added Q4: BD675, Package_TO_SOT_THT:TO-126-3_Vertical, F.Cu at (186.7, 119.4)
- added Q5: BD675, Package_TO_SOT_THT:TO-126-3_Vertical, F.Cu at (190.5, 105.4)
- added Q6: BD675, Package_TO_SOT_THT:TO-126-3_Vertical, F.Cu at (190.5, 114.3)
- added R6: 200, Resistor_SMD:R_0603_1608Metric_Pad1.05x0.95mm_HandSolder, F.Cu at (155.3, 109.2)
- added U3: LTV-845, Package_DIP:DIP-16_W7.62mm, F.Cu at (149.9, 111.8)
- R1, R2, R3, R4: value 330 -> 200; footprint Resistor_THT:R_Axial_DIN0207_L6.3mm_D2.5mm_P10.16mm_Horizontal -> Resistor_SMD:R_0603_1608Metric_Pad1.05x0.95mm_HandSolder
- R5: value 150 -> 200; footprint Resistor_THT:R_Axial_DIN0207_L6.3mm_D2.5mm_P10.16mm_Horizontal -> Resistor_SMD:R_0603_1608Metric_Pad1.05x0.95mm_HandSolder
- U2: value MOC3041M -> LTV-825; footprint Package_DIP:DIP-6_W7.62mm -> Package_DIP:DIP-8_W7.62mm
- moved R2 21.5 mm to (145.7, 109.2), turned to 0 degrees
- moved R1 18.2 mm to (150.7, 109.2), turned to 0 degrees
- moved U2 18.0 mm to (161.3, 111.8)
- moved R3 17.1 mm to (141.0, 109.2), turned to 0 degrees
- moved R4 16.8 mm to (136.3, 109.2), turned to 0 degrees
- moved R5 13.6 mm to (159.6, 109.2)
Connections:
- net Net-(J1+1-Pad1) renamed +5V
- J1+1 pad 2: Net-(J1+1-Pad2) -> GND
- J1-1 pad 2: Net-(J1+1-Pad2) -> GND
- JP1 pad 1: Net-(J1+1-Pad2) -> GND
- JP2 pad 1: Net-(J1+1-Pad2) -> GND
- JP3 pad 1: Net-(J1+1-Pad2) -> GND
- U1 pad 14: Net-(J1+1-Pad2) -> GND
- U1 pad 2: Net-(R5-Pad1) -> Net-(R6-Pad1)
- U1 pad 3: Net-(U1-Pad3) -> Net-(R5-Pad1)
- U2 pad 2: Net-(J1+1-Pad2) -> GND
- U2 pad 4: Net-(J4-Pad2) -> GND
Routing:
- net Net-(J2-Pad1): track 0.00 -> 117.6 mm
- net Net-(Q3-Pad3): track 0.00 -> 95.5 mm
- net Net-(Q6-Pad3): track 0.00 -> 88.8 mm
- net Net-(J2-Pad5): track 0.00 -> 82.7 mm
- net Net-(Q4-Pad3): track 0.00 -> 81.1 mm
- net GND: track 0.00 -> 68.8 mm
- net Net-(J2-Pad3): track 0.00 -> 68.0 mm
- net Net-(J1-Pad5): track 0.00 -> 61.1 mm
- net Net-(D6-Pad1): track 0.00 -> 58.8 mm
- net Net-(Q2-Pad3): track 0.00 -> 57.4 mm
- net Net-(J1-Pad3): track 4.98 -> 62.1 mm
- net Net-(Q5-Pad3): track 0.00 -> 56.4 mm
- net Net-(J1+1-Pad2): track 56.2 -> 0.00 mm
- net Net-(J1-Pad1): track 0.00 -> 55.8 mm
- net Net-(D4-Pad1): track 0.00 -> 50.5 mm
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Other:
- board size 48.3 x 40.6 mm -> 64.8 x 40.6 mm
- board text added: "Opto-Adapter ©2021 Dominik Föhl"
- board text removed: "Multiplex Adapter ©2020 Dominik Föhl"
