File: PCB/Belegterkennung/Belegterkennung.kicad_pcb (KiCad board)
At the start: 2 copper layers, 59.7 x 43.2 mm, 34 parts, among them J1 Conn_01x02, J3 Conn_01x04, J4 Conn_01x08, U1 LTV-844

Commit message: Added new PCB and updated older ones.
Parts:
- R1, R2, R3, R4: value 10k -> 3,7k
Routing:
- net /RM4: track 72.2 -> 95.3 mm
- net /RM3: track 89.2 -> 84.6 mm
- net /RM1: track 113.6 -> 115.6 mm
- net Net-(D7-K): track 4.12 -> 5.23 mm
- net Net-(D15-A): track 4.12 -> 5.23 mm
- net AC: track 47.4 -> 47.1 mm, vias 0 -> 1
Other:
- board text added: "Belegterkennung V2 ©2024 Dominik Föhl"
- board text removed: "Belegterkennung V1 ©2024 Dominik Föhl"
